Commit message: added inertial tags, now showing in gazebo

File: urdf/nefive-unity.urdf (robot description, URDF)
Before this commit: robot nefive, 39 links, 38 joints
Links:
- link arms: mass None -> 0.18
- link chest_box: mass None -> 0.18
- link front_left_wheel: mass None -> 0.18
- link front_right_wheel: mass None -> 0.18
- link head: mass None -> 0.18
- link head_pan: mass None -> 0.18
- link head_tilt: mass None -> 0.18
- link left_arm: mass None -> 0.18
- link left_elbow: mass None -> 0.18
- link left_eye_inner: mass None -> 0.18
- link left_eye_ring: mass None -> 0.18
- link left_forearm: mass None -> 0.18
- link left_hand: mass None -> 0.18
- link left_shoulder_pan: mass None -> 0.18
- link left_shoulder_rotate: mass None -> 0.18
- link left_shoulder_tilt: mass None -> 0.18
- link left_wrist_pan: mass None -> 0.18
- link left_wrist_roll: mass None -> 0.18
- link left_wrist_tilt: mass None -> 0.18
- link lower_torso: mass None -> 0.18
- link rear_left_idler: mass None -> 0.18
- link rear_left_wheel: mass None -> 0.18
- link rear_right_idler: mass None -> 0.18
- link rear_right_wheel: mass None -> 0.18
- link right_arm: mass None -> 0.18
- link right_elbow: mass None -> 0.18
- link right_eye_inner: mass None -> 0.18
- link right_eye_ring: mass None -> 0.18
- link right_forearm: mass None -> 0.18
- link right_hand: mass None -> 0.18
- link right_shoulder_pan: mass None -> 0.18
- link right_shoulder_rotate: mass None -> 0.18
- link right_shoulder_tilt: mass None -> 0.18
- link right_wrist_pan: mass None -> 0.18
- link right_wrist_roll: mass None -> 0.18
- link right_wrist_tilt: mass None -> 0.18
- link upper_torso: mass None -> 0.18

Commit message: added dummy inertias to get it running in Gazebo

File: urdf/nefive-unity.urdf (robot description, URDF)
Before this commit: robot nefive, 39 links, 38 joints
Links:
- link arms: mass None -> 0.18; geometry collision cylinder length=0 radius=0; visual cylinder length=0 radius=0
- link base_link: mass None -> 0.18
- link chest_box: mass None -> 0.18
- link eyes: mass None -> 0.18; geometry collision cylinder length=0 radius=0; visual cylinder length=0 radius=0
- link front_left_wheel: mass None -> 0.18
- link front_right_wheel: mass None -> 0.18
- link head: mass None -> 0.18
- link head_pan: mass None -> 0.18
- link head_tilt: mass None -> 0.18
- link left_arm: mass None -> 0.18; geometry collision cylinder length=0 radius=0; visual cylinder length=0 radius=0
- link left_elbow: mass None -> 0.18; geometry collision cylinder length=0 radius=0; visual cylinder length=0 radius=0
- link left_eye_inner: mass None -> 0.18
- link left_eye_ring: mass None -> 0.18
- link left_forearm: mass None -> 0.18
- link left_hand: mass None -> 0.18
- link left_shoulder_pan: mass None -> 0.18
- link left_shoulder_rotate: mass None -> 0.18
- link left_shoulder_tilt: mass None -> 0.18
- link left_wrist_pan: mass None -> 0.18
- link left_wrist_roll: mass None -> 0.18
- link left_wrist_tilt: mass None -> 0.18
- link lower_torso: mass None -> 0.18
- link rear_left_idler: mass None -> 0.18
- link rear_left_wheel: mass None -> 0.18
- link rear_right_idler: mass None -> 0.18
- link rear_right_wheel: mass None -> 0.18
- link right_arm: mass None -> 0.18; geometry collision cylinder length=0 radius=0; visual cylinder length=0 radius=0
- link right_elbow: mass None -> 0.18; geometry collision cylinder length=0 radius=0; visual cylinder length=0 radius=0
- link right_eye_inner: mass None -> 0.18
- link right_eye_ring: mass None -> 0.18
- link right_forearm: mass None -> 0.18
- link right_hand: mass None -> 0.18
- link right_shoulder_pan: mass None -> 0.18
- link right_shoulder_rotate: mass None -> 0.18
- link right_shoulder_tilt: mass None -> 0.18
- link right_wrist_pan: mass None -> 0.18
- link right_wrist_roll: mass None -> 0.18
- link right_wrist_tilt: mass None -> 0.18
- link upper_torso: mass None -> 0.18

Commit message: setting mass to negligible for now

File: urdf/nefive-unity.urdf (robot description, URDF)
Before this commit: robot nefive, 39 links, 38 joints
Links:
- link arms: mass 0.18 -> 0.001
- link base_link: mass 0.18 -> 0.001
- link chest_box: mass 0.18 -> 0.001
- link eyes: mass 0.18 -> 0.001
- link front_left_wheel: mass 0.18 -> 0.001
- link front_right_wheel: mass 0.18 -> 0.001
- link head: mass 0.18 -> 0.001
- link head_pan: mass 0.18 -> 0.001
- link head_tilt: mass 0.18 -> 0.001
- link left_arm: mass 0.18 -> 0.001
- link left_elbow: mass 0.18 -> 0.001
- link left_eye_inner: mass 0.18 -> 0.001
- link left_eye_ring: mass 0.18 -> 0.001
- link left_forearm: mass 0.18 -> 0.001
- link left_hand: mass 0.18 -> 0.001
- link left_shoulder_pan: mass 0.18 -> 0.001
- link left_shoulder_rotate: mass 0.18 -> 0.001
- link left_shoulder_tilt: mass 0.18 -> 0.001
- link left_wrist_pan: mass 0.18 -> 0.001
- link left_wrist_roll: mass 0.18 -> 0.001
- link left_wrist_tilt: mass 0.18 -> 0.001
- link lower_torso: mass 0.18 -> 0.001
- link rear_left_idler: mass 0.18 -> 0.001
- link rear_left_wheel: mass 0.18 -> 0.001
- link rear_right_idler: mass 0.18 -> 0.001
- link rear_right_wheel: mass 0.18 -> 0.001
- link right_arm: mass 0.18 -> 0.001
- link right_elbow: mass 0.18 -> 0.001
- link right_eye_inner: mass 0.18 -> 0.001
- link right_eye_ring: mass 0.18 -> 0.001
- link right_forearm: mass 0.18 -> 0.001
- link right_hand: mass 0.18 -> 0.001
- link right_shoulder_pan: mass 0.18 -> 0.001
- link right_shoulder_rotate: mass 0.18 -> 0.001
- link right_shoulder_tilt: mass 0.18 -> 0.001
- link right_wrist_pan: mass 0.18 -> 0.001
- link right_wrist_roll: mass 0.18 -> 0.001
- link right_wrist_tilt: mass 0.18 -> 0.001
- link upper_torso: mass 0.18 -> 0.001

Commit message: added camera links

File: urdf/nefive-unity.urdf (robot description, URDF)
Before this commit: robot nefive, 39 links, 38 joints
Links:
- added link left_camera, mass 0.001
- added link right_camera, mass 0.001
Joints:
- added joint left_eye_inner_left_camera_joint: type fixed, parent left_eye_inner, child left_camera
- added joint right_eye_inner_right_camera_joint: type fixed, parent right_eye_inner, child right_camera

Commit message: fixed the inverted wheel axes

File: urdf/nefive-unity.urdf (robot description, URDF)
Before this commit: robot nefive, 41 links, 40 joints
Joints:
- joint base_link_front_left_wheel_joint: axis 0 -1 0 -> 0 1 0
- joint base_link_front_right_wheel_joint: axis 0 -1 0 -> 0 1 0
- joint base_link_rear_left_idler_joint: axis 0 -1 0 -> 0 1 0
- joint base_link_rear_left_wheel_joint: axis 0 -1 0 -> 0 1 0
- joint base_link_rear_right_idler_joint: axis 0 -1 0 -> 0 1 0
- joint base_link_rear_right_wheel_joint: axis 0 -1 0 -> 0 1 0

Commit message: Fixed the issue with the elbows forward being missing

File: urdf/nefive-unity.urdf (robot description, URDF)
Before this commit: robot nefive, 41 links, 40 joints
Links:
- added link chassis, mass 0.001; collision box size=0.07 0.02 0.01; collision box size=0.07 0.02 0.01
- link base_link: mass 0.001 -> None; geometry 
- link left_elbow: geometry collision cylinder length=0.02 radius=0.0005; visual cylinder length=0.02 radius=0.0005
- link right_elbow: geometry collision cylinder length=0.02 radius=0.0005; visual cylinder length=0.02 radius=0.0005
Joints:
- added joint base_link_to_chassis: type fixed, parent base_link, child chassis
- joint base_link_front_left_wheel_joint: parent base_link -> chassis
- joint base_link_front_right_wheel_joint: parent base_link -> chassis
- joint base_link_lower_torso_joint: parent base_link -> chassis
- joint base_link_rear_left_idler_joint: parent base_link -> chassis
- joint base_link_rear_left_wheel_joint: parent base_link -> chassis
- joint base_link_rear_right_idler_joint: parent base_link -> chassis
- joint base_link_rear_right_wheel_joint: parent base_link -> chassis

Commit message: fixed the missing links in rviz

File: urdf/nefive-unity.urdf (robot description, URDF)
Before this commit: robot nefive, 42 links, 41 joints
Joints:
- joint base_link_rear_left_idler_joint: type continuous -> fixed
- joint base_link_rear_right_idler_joint: type continuous -> fixed

Commit message: Got the colouring working in Gazebo

File: urdf/nefive-unity.urdf (robot description, URDF)
Before this commit: robot nefive, 42 links, 41 joints
Links:
- added link upper_tracks, mass 1; collision box size=0.07 0.02 0.01; collision box size=0.07 0.02 0.01
- link chassis: geometry collision box size=0.104 0.147 0.068; visual box size=0.104 0.147 0.068
Joints:
- removed joint base_link_to_chassis
- added joint : type fixed, parent chassis, child upper_tracks
- added joint base_link_chassis_joint: type fixed, parent base_link, child chassis
- joint base_link_rear_left_idler_joint: axis 0 1 0 -> (none)
- joint base_link_rear_right_idler_joint: axis 0 1 0 -> (none)
- joint left_forearm_left_wrist_roll_joint: origin xyz=0.0683 -0.0025 0 rpy=0 4.712389 0 -> xyz=0.0683 -0.0025 0 rpy=0 4.712734 0
- joint lower_torso_upper_torso_joint: origin xyz=0 0 0.06 rpy=0 1.570796 0 -> xyz=0 0 0.06 rpy=0 1.570451 0
