Commit message: renamed the urdf

File: urdf/nefive.urdf (robot description, URDF)
Before this commit: robot nefive, 21 links, 20 joints
Links:
- removed link chest_box_link
- removed link eye_ring_inner_left_link
- removed link eye_ring_inner_right_link
- removed link eye_ring_left_link
- removed link eye_ring_right_link
- removed link head_link
- removed link left_forearm_link
- removed link left_hand_link
- removed link left_shoulder_link
- removed link left_upperarm_link
- removed link lowertorso_link
- removed link right_forearm_link
- removed link right_hand_link
- removed link right_shoulder_link
- removed link right_upperarm_link
- removed link roll_M0_idler_link
- removed link roll_M0_link
- removed link roll_M1_idler_link
- removed link roll_M1_link
- removed link uppertorso_link
- added link arms, mass 0.001
- added link chassis, mass 0.001; collision box size=0.104 0.147 0.068; visual box size=0.104 0.147 0.068
- added link chest_box, mass 0.001; collision box size=0.05 0.07 0.05; visual box size=0.05 0.07 0.05
- added link eyes, mass 0.001; collision cylinder length=0 radius=0; visual cylinder length=0 radius=0
- added link front_left_wheel, mass 0.001; collision cylinder length=0.02 radius=0.025; visual cylinder length=0.02 radius=0.025
- added link front_right_wheel, mass 0.001; collision cylinder length=0.02 radius=0.025; visual cylinder length=0.02 radius=0.025
- added link head, mass 0.001; collision box size=0.107 0.11 0.054; visual box size=0.107 0.11 0.054
- added link head_pan, mass 0.001; collision cylinder length=0.002 radius=0.02; visual cylinder length=0.002 radius=0.02
- added link head_tilt, mass 0.001; collision box size=0.04 0.04 0.001; visual box size=0.04 0.04 0.001
- added link left_arm, mass 0.001
- added link left_camera, mass 0.001
- added link left_elbow, mass 0.001; collision cylinder length=0.02 radius=0.0005; visual cylinder length=0.02 radius=0.0005
- added link left_eye_inner, mass 0.001; collision cylinder length=0.002 radius=0.01; visual cylinder length=0.002 radius=0.01
- added link left_eye_ring, mass 0.001; collision cylinder length=0.002 radius=0.02; visual cylinder length=0.002 radius=0.02
- added link left_forearm, mass 0.001; collision cylinder length=0.07 radius=0.005; visual cylinder length=0.07 radius=0.005
- added link left_hand, mass 0.001; visual box size=0.02 0.02 0.02
- added link left_shoulder_pan, mass 0.001; collision cylinder length=0.004 radius=0.0005; visual cylinder length=0.004 radius=0.0005
- added link left_shoulder_rotate, mass 0.001; collision cylinder length=-0.06 radius=0.005; collision cylinder length=0.004 radius=0.0005
- added link left_shoulder_tilt, mass 0.001; collision cylinder length=0.02 radius=0.0005; visual cylinder length=0.02 radius=0.0005
- added link left_wrist_pan, mass 0.001; collision cylinder length=0.01 radius=0.0005; visual cylinder length=0.01 radius=0.0005
- added link left_wrist_roll, mass 0.001; collision cylinder length=0.01 radius=0.0005; visual cylinder length=0.01 radius=0.0005
- added link left_wrist_tilt, mass 0.001; collision cylinder length=0.01 radius=0.0005; visual cylinder length=0.01 radius=0.0005
- added link lower_torso, mass 0.001; collision box size=0.015 0.06 0.06; visual box size=0.015 0.06 0.06
- added link rear_left_idler, mass 0.001; collision cylinder length=0.02 radius=0.025; visual cylinder length=0.02 radius=0.025
- added link rear_left_wheel, mass 0.001; collision cylinder length=0.02 radius=0.025; visual cylinder length=0.02 radius=0.025
- added link rear_right_idler, mass 0.001; collision cylinder length=0.02 radius=0.025; visual cylinder length=0.02 radius=0.025
- added link rear_right_wheel, mass 0.001; collision cylinder length=0.02 radius=0.025; visual cylinder length=0.02 radius=0.025
- added link right_arm, mass 0.001
- added link right_camera, mass 0.001
- added link right_elbow, mass 0.001; collision cylinder length=0.02 radius=0.0005; visual cylinder length=0.02 radius=0.0005
- added link right_eye_inner, mass 0.001; collision cylinder length=0.002 radius=0.01; visual cylinder length=0.002 radius=0.01
- added link right_eye_ring, mass 0.001; collision cylinder length=0.002 radius=0.02; visual cylinder length=0.002 radius=0.02
- added link right_forearm, mass 0.001; collision cylinder length=0.07 radius=0.005; visual cylinder length=0.07 radius=0.005
- added link right_hand, mass 0.001; visual box size=0.02 0.02 0.02
- added link right_shoulder_pan, mass 0.001; collision cylinder length=0.004 radius=0.0005; visual cylinder length=0.004 radius=0.0005
- added link right_shoulder_rotate, mass 0.001; collision cylinder length=-0.06 radius=0.005; collision cylinder length=0.004 radius=0.0005
- added link right_shoulder_tilt, mass 0.001; collision cylinder length=0.02 radius=0.0005; visual cylinder length=0.02 radius=0.0005
- added link right_wrist_pan, mass 0.001; collision cylinder length=0.01 radius=0.0005; visual cylinder length=0.01 radius=0.0005
- added link right_wrist_roll, mass 0.001; collision cylinder length=0.01 radius=0.0005; visual cylinder length=0.01 radius=0.0005
- added link right_wrist_tilt, mass 0.001; collision cylinder length=0.01 radius=0.0005; visual cylinder length=0.01 radius=0.0005
- added link upper_torso, mass 0.001; collision box size=0.015 0.06 0.06; visual box size=0.015 0.06 0.06
- added link upper_tracks, mass 1; collision box size=0.07 0.02 0.01; collision box size=0.07 0.02 0.01
- link base_link: geometry 
Joints:
- removed joint base_chest_box_fixed
- removed joint base_lowertorso_fixed
- removed joint chest_box_head_fixed
- removed joint chest_box_left_shoulder_fixed
- removed joint chest_box_right_shoulder_fixed
- removed joint head_eye_ring_inner_left_fixed
- removed joint head_eye_ring_inner_right_fixed
- removed joint head_eye_ring_left_fixed
- removed joint head_eye_ring_right_fixed
- removed joint left_forearm_hand_fixed
- removed joint left_shoulder_upperarm_fixed
- removed joint left_upperarm_forearm_fixed
- removed joint lowertorso_uppertorso_fixed
- removed joint right_forearm_hand_fixed
- removed joint right_shoulder_upperarm_fixed
- removed joint right_upperarm_forearm_fixed
- removed joint roll_joint_M0
- removed joint roll_joint_M0_idler
- removed joint roll_joint_M1
- removed joint roll_joint_M1_idler
- added joint : type fixed, parent chassis, child upper_tracks
- added joint arms_left_arm_joint: type fixed, parent arms, child left_arm, origin xyz=0 0.06 0 rpy=0 0 -3.141593
- added joint arms_right_arm_joint: type fixed, parent arms, child right_arm, origin xyz=0 -0.06 0
- added joint base_link_chassis_joint: type fixed, parent base_link, child chassis
- added joint base_link_front_left_wheel_joint: type continuous, parent chassis, child front_left_wheel, origin xyz=0.07 0.078 -0.022, axis 0 1 0
- added joint base_link_front_right_wheel_joint: type continuous, parent chassis, child front_right_wheel, origin xyz=0.07 -0.078 -0.022, axis 0 1 0
- added joint base_link_lower_torso_joint: type fixed, parent chassis, child lower_torso, origin xyz=-0.0241 0 0.0285 rpy=0 5.497787 0
- added joint base_link_rear_left_idler_joint: type fixed, parent chassis, child rear_left_idler, origin xyz=-0.0402 0.078 0.0271
- added joint base_link_rear_left_wheel_joint: type continuous, parent chassis, child rear_left_wheel, origin xyz=-0.07 0.078 -0.022, axis 0 1 0
- added joint base_link_rear_right_idler_joint: type fixed, parent chassis, child rear_right_idler, origin xyz=-0.0402 -0.078 0.0271
- added joint base_link_rear_right_wheel_joint: type continuous, parent chassis, child rear_right_wheel, origin xyz=-0.07 -0.078 -0.022, axis 0 1 0
- added joint chest_box_arms_joint: type fixed, parent chest_box, child arms, origin xyz=0.025 0 0.075
- added joint chest_box_head_pan_joint: type revolute, parent chest_box, child head_pan, origin xyz=0.025 0 0.0819, axis 0 0 1, limit lower=-0.785398 upper=0.785398 effort=1000 velocity=1000
- added joint eyes_left_eye_ring_joint: type fixed, parent eyes, child left_eye_ring, origin xyz=0 0.03 0
- added joint eyes_right_eye_ring_joint: type fixed, parent eyes, child right_eye_ring, origin xyz=0 -0.03 0
- added joint head_eyes_joint: type fixed, parent head, child eyes, origin xyz=0.05 0 0.03
- added joint head_pan_head_tilt_joint: type revolute, parent head_pan, child head_tilt, origin xyz=0 0 0.035, axis 0 -1 0, limit lower=-0.785398 upper=0.785398 effort=1000 velocity=1000
- added joint head_tilt_head_joint: type fixed, parent head_tilt, child head
- added joint left_arm_left_shoulder_tilt_joint: type revolute, parent left_arm, child left_shoulder_tilt, origin rpy=0 5.497787 0, axis 1 0 0, limit lower=-0.610865 upper=0.436332 effort=1000 velocity=1000
- added joint left_elbow_left_forearm_joint: type revolute, parent left_elbow, child left_forearm, origin xyz=0.01 0 0.0025 rpy=-3.141593 0.785398 -3.141593, axis 0 -1 0, limit lower=0 upper=0 effort=1000 velocity=1000
- added joint left_eye_inner_left_camera_joint: type fixed, parent left_eye_inner, child left_camera
- added joint left_eye_ring_left_eye_inner_joint: type fixed, parent left_eye_ring, child left_eye_inner
- added joint left_forearm_left_wrist_roll_joint: type revolute, parent left_forearm, child left_wrist_roll, origin xyz=0.0683 -0.0025 0 rpy=0 4.712734 0, axis 0 0 1, limit lower=-1.570796 upper=1.570796 effort=1000 velocity=1000
- added joint left_shoulder_pan_left_shoulder_rotate_joint: type revolute, parent left_shoulder_pan, child left_shoulder_rotate, origin xyz=0 -0.0048 0 rpy=0 5.497787 0, axis 1 0 0, limit lower=-1.570796 upper=1.570796 effort=1000 velocity=1000
- added joint left_shoulder_rotate_left_elbow_joint: type revolute, parent left_shoulder_rotate, child left_elbow, origin xyz=0.075 0 0, axis 0 -1 0, limit lower=0 upper=0 effort=1000 velocity=1000
- added joint left_shoulder_tilt_left_shoulder_pan_joint: type revolute, parent left_shoulder_tilt, child left_shoulder_pan, origin xyz=0 -0.001 0 rpy=-3.141593 0.785398 -3.141593, axis 0 -1 0, limit lower=-1.570796 upper=1.570796 effort=1000 velocity=1000
- added joint left_wrist_pan_left_hand_joint: type fixed, parent left_wrist_pan, child left_hand, origin xyz=0.012 0 0
- added joint left_wrist_roll_left_wrist_tilt_joint: type revolute, parent left_wrist_roll, child left_wrist_tilt, origin xyz=0 0 -0.00636 rpy=0 1.570796 -4.712389, axis 0 0 1, limit lower=-0.785398 upper=0.785398 effort=1000 velocity=1000
- added joint left_wrist_tilt_left_wrist_pan_joint: type revolute, parent left_wrist_tilt, child left_wrist_pan, origin xyz=0.002 0 0 rpy=-4.712389 0 0, axis 0 0 1, limit lower=-0.785398 upper=0.785398 effort=1000 velocity=1000
- added joint lower_torso_upper_torso_joint: type fixed, parent lower_torso, child upper_torso, origin xyz=0 0 0.06 rpy=0 1.570451 0
- added joint right_arm_right_shoulder_tilt_joint: type revolute, parent right_arm, child right_shoulder_tilt, origin rpy=0 0.785398 0, axis 1 0 0, limit lower=-0.610865 upper=0.436332 effort=1000 velocity=1000
- added joint right_elbow_right_forearm_joint: type revolute, parent right_elbow, child right_forearm, origin xyz=0.01 0 0.0025 rpy=-3.141593 5.497787 -3.141593, axis 0 -1 0, limit lower=0 upper=0 effort=1000 velocity=1000
- added joint right_eye_inner_right_camera_joint: type fixed, parent right_eye_inner, child right_camera
- added joint right_eye_ring_right_eye_inner_joint: type fixed, parent right_eye_ring, child right_eye_inner
- added joint right_forearm_right_wrist_roll_joint: type revolute, parent right_forearm, child right_wrist_roll, origin xyz=0.0683 -0.0025 0 rpy=0 4.712389 0, axis 0 0 1, limit lower=-1.570796 upper=1.570796 effort=1000 velocity=1000
- added joint right_shoulder_pan_right_shoulder_rotate_joint: type revolute, parent right_shoulder_pan, child right_shoulder_rotate, origin xyz=0 -0.0048 0 rpy=0 0.785398 0, axis 1 0 0, limit lower=-1.570796 upper=1.570796 effort=1000 velocity=1000
- added joint right_shoulder_rotate_right_elbow_joint: type revolute, parent right_shoulder_rotate, child right_elbow, origin xyz=0.075 0 0, axis 0 -1 0, limit lower=0 upper=0 effort=1000 velocity=1000
- added joint right_shoulder_tilt_right_shoulder_pan_joint: type revolute, parent right_shoulder_tilt, child right_shoulder_pan, origin xyz=0 -0.001 0 rpy=0 0.785398 0, axis 0 -1 0, limit lower=-1.570796 upper=1.570796 effort=1000 velocity=1000
- added joint right_wrist_pan_right_hand_joint: type fixed, parent right_wrist_pan, child right_hand, origin xyz=0.012 0 0
- added joint right_wrist_roll_right_wrist_tilt_joint: type revolute, parent right_wrist_roll, child right_wrist_tilt, origin xyz=0 0 -0.00636 rpy=0 1.570796 -4.712389, axis 0 0 1, limit lower=-0.785398 upper=0.785398 effort=1000 velocity=1000
- added joint right_wrist_tilt_right_wrist_pan_joint: type revolute, parent right_wrist_tilt, child right_wrist_pan, origin xyz=0.002 0 0 rpy=-4.712389 0 0, axis 0 0 1, limit lower=-0.785398 upper=0.785398 effort=1000 velocity=1000
- added joint upper_torso_chest_box_joint: type fixed, parent upper_torso, child chest_box, origin xyz=0.0305 0 0.0269 rpy=0 5.497787 0
